Commit message: additional changes

File: auto_ws/src/rover_assembly_urdf/urdf/Rover Assembly URDF.urdf (robot description, URDF)
Before this commit: robot Rover Assembly URDF, 5 links, 4 joints
Links:
- added link camera_link; visual box size=0.025 0.09 0.025
Joints:
- added joint camera_joint: type fixed, parent base_link, child camera_link, origin xyz=0.3 0 0.1 rpy=0 0 0

Commit message: update for simulations

File: auto_ws/src/rover_assembly_urdf/urdf/Rover Assembly URDF.urdf (robot description, URDF)
Before this commit: robot Rover Assembly URDF, 6 links, 5 joints
Links:
- link base_link: geometry collision mesh filename=package://rover_assembly_urdf/meshes/base_link.STL; visual mesh filename=package://rover_assembly_urdf/meshes/base_link.STL
- link front_left_wheel: geometry collision mesh filename=package://rover_assembly_urdf/meshes/front_left_wheel.STL; visual mesh filename=package://rover_assembly_urdf/meshes/front_left_wheel.STL
- link front_right_wheel: geometry collision mesh filename=package://rover_assembly_urdf/meshes/front_right_wheel.STL; visual mesh filename=package://rover_assembly_urdf/meshes/front_right_wheel.STL
- link rear_left_wheel: geometry collision mesh filename=package://rover_assembly_urdf/meshes/rear_left_wheel.STL; visual mesh filename=package://rover_assembly_urdf/meshes/rear_left_wheel.STL
- link rear_right_wheel: geometry collision mesh filename=package://rover_assembly_urdf/meshes/rear_right_wheel.STL; visual mesh filename=package://rover_assembly_urdf/meshes/rear_right_wheel.STL
